File: SXMtoPCIe/SXMtoPCIe.kicad_sch (KiCad schematic)
At the start: 36 parts, among them J1 Bus_PCI_Express_x16, J2 74221-101LF, J3 74221-101LF

Commit message: save
Parts:
- added D2: BAT54J, Diode_SMD:D_SOD-123, symbol Diode:BAT54J
- added R1: 10k, Resistor_SMD:R_0402_1005Metric, symbol Device:R
Connections:
- net GND: now also J2.A1, J2.A10, J2.A13, J2.A14, J2.A17, J2.A19, J2.A4, J2.A7, J2.B11, J2.B14, J2.B15, J2.B18, J2.B19, J2.B3, J2.B6, J2.B7, J2.B8, J2.C1, J2.C10, J2.C13, J2.C14, J2.C17, J2.C19, J2.C4, J2.C7, J2.D11, J2.D14, J2.D15, J2.D18, J2.D19, J2.D3, J2.D6, J2.D7, J2.D8, J2.E1, J2.E10, J2.E11, J2.E12, J2.E13, J2.E14, J2.E15, J2.E16, J2.E17, J2.E19, J2.E2, J2.E3, J2.E4, J2.E5, J2.E6, J2.E8, J2.E9, J2.F1, J2.F10, J2.F11, J2.F12, J2.F13, J2.F14, J2.F15, J2.F16, J2.F17, J2.F19, J2.F2, J2.F3, J2.F4, J2.F5, J2.F6, J2.F8, J2.F9, J2.G11, J2.G14, J2.G15, J2.G18, J2.G19, J2.G3, J2.G6, J2.G7, J2.G8, J2.H1, J2.H10, J2.H13, J2.H14, J2.H17, J2.H4, J2.H7, J2.J11, J2.J14, J2.J15, J2.J18, J2.J19, J2.J3, J2.J6, J2.J7, J2.J8, J2.K1, J2.K10, J2.K13, J2.K14, J2.K17, J2.K4, J2.K7
- net PER0_N: now also J2.A3
- net PER0_P: now also J2.A2
- net PER10_N: now also J2.C9
- net PER10_P: now also J2.C8
- net PER11_N: now also J2.D10
- net PER11_P: now also J2.D9
- net PER12_N: now also J2.A12
- net PER12_P: now also J2.A11
- net PER13_N: now also J2.C12
- net PER13_P: now also J2.C11
- net PER14_N: now also J2.D13
- net PER14_P: now also J2.D12
- net PER15_N: now also J2.B13
- net PER15_P: now also J2.B12
- net PER1_N: now also J2.B2
- net PER1_P: now also J2.B1
- net PER2_N: now also J2.D2
- net PER2_P: now also J2.D1
- net PER3_N: now also J2.C3
- net PER3_P: now also J2.C2
- net PER4_N: now also J2.B5
- net PER4_P: now also J2.B4
- net PER5_N: now also J2.D5
- net PER5_P: now also J2.D4
- net PER6_N: now also J2.C6
- net PER6_P: now also J2.C5
- net PER7_N: now also J2.A6
- net PER7_P: now also J2.A5
- net PER8_N: now also J2.A9
- net PER8_P: now also J2.A8
- net PER9_N: now also J2.B10
- net PER9_P: now also J2.B9
- net at J1.A1 (~{PRSNT1}): now also J1.B81 (~{PRSNT2})
- net /PERST: now reaches J1.A11 (~{PERST})
- net /PERST: now also J2.E18
- net REFCLK+: now reaches J1.A13 (REFCLK+)
- net REFCLK+: now also J2.E7
- net REFCLK-: now reaches J1.A14 (REFCLK-)
- net REFCLK-: now also J2.F7
- net PET0_P: now reaches J1.B14 (PETp0)
- net PET0_P: now also J2.G1
- net PET0_N: now reaches J1.B15 (PETn0)
- net PET0_N: now also J2.G2
- net PET1_P: now reaches J1.B19 (PETp1)
- net PET1_P: now also J2.H2
- net PET1_N: now reaches J1.B20 (PETn1)
- net PET1_N: now also J2.H3
- net PET2_P: now reaches J1.B23 (PETp2)
- net PET2_P: now also J2.J1
- net PET2_N: now reaches J1.B24 (PETn2)
- net PET2_N: now also J2.J2
- net PET3_P: now reaches J1.B27 (PETp3)
- net PET3_P: now also J2.K2
- net PET3_N: now reaches J1.B28 (PETn3)
- net PET3_N: now also J2.K3
- net PET4_P: now reaches J1.B33 (PETp4)
- net PET4_P: now also J2.G4
- net PET4_N: now reaches J1.B34 (PETn4)
- net PET4_N: now also J2.G5
- net PET5_P: now reaches J1.B37 (PETp5)
- net PET5_P: now also J2.J4
- net PET5_N: now reaches J1.B38 (PETn5)
- net PET5_N: now also J2.J5
- net PET6_P: now reaches J1.B41 (PETp6)
- net PET6_P: now also J2.K5
- net PET6_N: now reaches J1.B42 (PETn6)
- net PET6_N: now also J2.K6
- net PET7_P: now reaches J1.B45 (PETp7)
- net PET7_P: now also J2.H5
- net PET7_N: now reaches J1.B46 (PETn7)
- net PET7_N: now also J2.H6
- net PET8_P: now reaches J1.B50 (PETp8)
- net PET8_P: now also J2.G9
- net PET8_N: now reaches J1.B51 (PETn8)
- net PET8_N: now also J2.G10
- net PET9_P: now reaches J1.B54 (PETp9)
- net PET9_P: now also J2.H8
- net PET9_N: now reaches J1.B55 (PETn9)
- net PET9_N: now also J2.H9
- net PET10_P: now reaches J1.B58 (PETp10)
- net PET10_P: now also J2.K8
- net PET10_N: now reaches J1.B59 (PETn10)
- net PET10_N: now also J2.K9
- net PET11_P: now reaches J1.B62 (PETp11)
- net PET11_P: now also J2.J9
- net PET11_N: now reaches J1.B63 (PETn11)
- net PET11_N: now also J2.J10
- net PET12_P: now reaches J1.B66 (PETp12)
- net PET12_P: now also J2.H11
- net PET12_N: now reaches J1.B67 (PETn12)
- net PET12_N: now also J2.H12
- net PET13_P: now reaches J1.B70 (PETp13)
- net PET13_P: now also J2.K11
- net PET13_N: now reaches J1.B71 (PETn13)
- net PET13_N: now also J2.K12
- net PET14_P: now reaches J1.B74 (PETp14)
- net PET14_P: now also J2.J12
- net PET14_N: now reaches J1.B75 (PETn14)
- net PET14_N: now also J2.J13
- net PET15_P: now reaches J1.B78 (PETp15)
- net PET15_P: now also J2.G12
- net PET15_N: now reaches J1.B79 (PETn15)
- net PET15_N: now also J2.G13
- net K18: now reaches J2.K18
- net K18: now also D2.1 (K)
- net K19: now reaches J2.K19
- net K19: now also R1.1
- new net +3V3: D2.2 (A), R1.2
Other:
- note added: "Protection Circuit (??)"
- company: (none) -> Benchoff
- title: (none) -> SXM2 PCIe Adapter
