File: SXMtoPCIe/SXMtoPCIe.kicad_sch (KiCad schematic)
At the start: 38 parts, among them J1 Bus_PCI_Express_x16, J2 74221-101LF, J3 74221-101LF

Commit message: Adds refs, partial routing progress
Parts:
- J2, J3: footprint SXM-AMP:AMPHENOL_74221-101LF -> 74221-101LF:AMPHENOL_74221-101LF

Commit message: Progress on power
Parts:
- added C33, C34, C35, C36: 470uF, symbol Device:C_Polarized_US
Connections:
- new net +12HPWR: C33.1, C34.1, C35.1, C36.1
- new net GNDHPWR: C33.2, C34.2, C35.2, C36.2
Other:
- note added: "https://www.mouser.co.uk/en/ProductDetail/Molex/45586-0005"

Commit message: Power routing more or less complete
Parts:
- added J4, J5: Molex_45586-0005, CONN_455860000-SD_MOL, symbol 45586-0005:455860005
- C1, C10, C11, C12, C13, C14, C15, C16, C17, C18, C19, C2, C20, C21, C22, C23, C24, C25, C26, C27, C28, C29, C3, C30, C31, C32, C4, C5, C6, C7, C8, C9: footprint Capacitor_SMD:C_0201_0603Metric -> Capacitor_SMD:C_0201_0603Metric_Pad0.64x0.40mm_HandSolder
- C33, C34, C35, C36: footprint (none) -> Capacitor_SMD:CP_Elec_6.3x7.7
- R1: footprint Resistor_SMD:R_0402_1005Metric -> Resistor_SMD:R_0402_1005Metric_Pad0.72x0.64mm_HandSolder
Connections:
- net +12V is gone; now on net +12VPCI: J2.A22, J2.A23, J2.A25, J2.A26, J2.A28, J2.A29, J2.A31, J2.A32, J2.A34, J2.A35, J2.A37, J2.A38, J2.A40, J2.B22, J2.B23, J2.B25, J2.B26, J2.B28, J2.B29, J2.B31, J2.B32, J2.B34, J2.B35, J2.B37, J2.B38, J2.B40, J2.C22, J2.C23, J2.C25, J2.C26, J2.C28, J2.C29, J2.C31, J2.C32, J2.C34, J2.C35, J2.C37, J2.C38, J2.C40, J2.D22, J2.D23, J2.D25, J2.D26, J2.D28, J2.D29, J2.D31, J2.D32, J2.D34, J2.D35, J2.D37, J2.D38, J2.D40, J2.E22, J2.E23, J2.E25, J2.E26, J2.E28, J2.E29, J2.E31, J2.E32, J2.E34, J2.E35, J2.E37, J2.E38, J2.E40, J2.F22, J2.F23, J2.F25, J2.F26, J2.F28, J2.F29, J2.F31, J2.F32, J2.F34, J2.F35, J2.F37, J2.F38, J2.F40, J2.G22, J2.G23, J2.G25, J2.G26, J2.G28, J2.G29, J2.G31, J2.G32, J2.G34, J2.G35, J2.G37, J2.G38, J2.G40, J2.H22, J2.H23, J2.H25, J2.H26, J2.H28, J2.H29, J2.H31, J2.H32, J2.H34, J2.H35, J2.H37, J2.H38, J2.H40, J2.J22, J2.J23, J2.J25, J2.J26, J2.J28, J2.J29, J2.J31, J2.J32, J2.J34, J2.J35, J2.J37, J2.J38, J2.J40, J2.K22, J2.K23, J2.K25, J2.K26, J2.K28, J2.K29, J2.K31, J2.K32, J2.K34, J2.K35, J2.K37, J2.K38, J2.K40
- net GNDHPWR is gone; now on net GND: C33.2, C34.2, C35.2, C36.2
- net GND: now also J4.4, J4.5, J4.6, J4.7, J4.8, J5.4, J5.5, J5.6, J5.7, J5.8
- net +12HPWR renamed +12VPCI
- net +12VPCI: now also J4.1, J4.2, J4.3, J5.1, J5.2, J5.3
Other:
- note added: "300W Power Delivery"
- note removed: "https://www.mouser.co.uk/en/ProductDetail/Molex/45586-0005"
- moved on the sheet: C1, C10, C11, C12, C13, C14, C15, C16, C17, C18, C19, C2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

Commit message: Mounting holes, finishing touches
Parts:
- added H1, H2, H3, H4: Bracket, MountingHole:MountingHole_3.2mm_M3_Pad_Via, symbol Mechanical:MountingHole_Pad
Connections:
- net +3V3: now also J1.A10 (+3.3V), J1.A9 (+3.3V), J1.B8 (+3.3V)
- net GND: now also H1.1, H2.1, H3.1, H4.1
- net +12V: now reaches J1.A2 (+12V), J1.A3 (+12V), J1.B1 (+12V), J1.B2 (+12V), J1.B3 (+12V)
