File: SXMtoPCIe/_autosave-SXMtoPCIe.kicad_pcb (KiCad board)
At the start: 4 copper layers, 172.5 x 111.3 mm, 38 parts, among them J1 Bus_PCI_Express_x16, J2 74221-101LF, J3 74221-101LF

Commit message: save
Routing:
- net PER7_P: track 0.88 -> 18.1 mm, vias 0 -> 1
- net PER7_N: track 0.88 -> 18.0 mm, vias 0 -> 1
- net PER0_N: track 0.35 -> 7.19 mm, vias 0 -> 1
- net PER0_P: track 0.35 -> 6.02 mm, vias 0 -> 1
- net PER1_N: track 0.35 -> 4.65 mm, vias 0 -> 1
- net PER2_N: track 0.00 -> 4.05 mm, vias 0 -> 1
- net PER1_P: track 0.35 -> 3.53 mm, vias 0 -> 1
- net PER2_P: track 0.00 -> 2.72 mm, vias 0 -> 1
- net PER4_N: track 1.08 -> 1.96 mm, vias 0 -> 1
- net PER4_P: track 1.01 -> 1.66 mm, vias 0 -> 1
